Commit message: - Fixed path ofr meshes in panda.urdf - Added CMakeLists.txt in resources for installation

File: resources/robots/panda/panda.urdf (robot description, URDF)
Before this commit: robot fp3, 10 links, 9 joints
Links:
- link fp3_link0: geometry collision cylinder length=0.03 radius=0.09; collision sphere radius=0.09
- link fp3_link1: geometry collision cylinder length=0.2830 radius=0.09; collision sphere radius=0.09
- link fp3_link2: geometry collision cylinder length=0.12 radius=0.09; collision sphere radius=0.09
- link fp3_link3: geometry collision cylinder length=0.15 radius=0.09; collision sphere radius=0.09
- link fp3_link4: geometry collision cylinder length=0.12 radius=0.09; collision sphere radius=0.09
- link fp3_link5: geometry collision cylinder length=0.1 radius=0.09; collision cylinder length=0.14 radius=0.055
- link fp3_link6: geometry collision cylinder length=0.08 radius=0.08; collision sphere radius=0.08
- link fp3_link7: geometry collision cylinder length=0.14 radius=0.07; collision sphere radius=0.07
