Commit message: Added example convex hull with go2

File: resources/robots/go2/go2.urdf (robot description, URDF)
Before this commit: robot go2_description, 42 links, 41 joints
Links:
- added link base_link
- added link world
Joints:
- added joint base_link_frame: type fixed, parent base, child base_link
- added joint reference: type floating, parent world, child base
